File: stm32f401nucl/piko_stm32f4nucl/piko_stm32f4nucl.kicad_pcb (KiCad board)
At the start: 2 copper layers, 35 parts, among them J1 Micro_SD_Card_Det, U1 NUCLEO-64

Commit message: progress nucleo board
Parts:
- moved D-ANS1 16.6 mm to (122.3, 124.7)
- moved C1 16.6 mm to (66.4, 131.2)
- moved R2 16.6 mm to (121.3, 133.6)
- moved D-AMPL1 16.6 mm to (145.6, 125.3)
- moved D-AMPL2 16.6 mm to (148.0, 125.3)
- moved D-AMPL4 16.6 mm to (153.0, 125.5)
- moved D-AMPL5 16.6 mm to (155.2, 125.5)
- moved D-FREQ1 16.6 mm to (145.6, 111.3)
- moved D-FREQ2 16.6 mm to (148.0, 111.4)
- moved D-FREQ3 16.6 mm to (150.4, 111.4)
- moved D-FREQ4 16.6 mm to (152.8, 111.4)
- moved R-AMPL1 16.6 mm to (141.3, 126.2)
- moved R-ANS1 16.6 mm to (82.9, 127.3)
- moved R-FREQ1 16.6 mm to (141.5, 110.3)
- moved R-GAIN1 16.6 mm to (67.9, 77.8)
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Routing:
- net VDD: track 92.3 -> 400.2 mm, vias 3 -> 9
- net /LRC: track 0.00 -> 177.0 mm, vias 0 -> 2
- net GND: track 188.4 -> 319.8 mm, vias 1 -> 4
- net /BCLK: track 0.00 -> 124.2 mm, vias 0 -> 2
- net /LED_M3: track 0.00 -> 65.9 mm, vias 0 -> 1
- net /RX: track 0.00 -> 52.6 mm, vias 0 -> 2
- net /LED_M1: track 0.00 -> 46.5 mm, vias 0 -> 1
- net /LED_M5: track 0.00 -> 46.4 mm, vias 0 -> 1
- net /LED_ANS_FALSE: track 3.90 -> 49.6 mm
- net /LED_M2: track 0.00 -> 44.9 mm, vias 0 -> 3
- net /TX: track 0.00 -> 42.4 mm
- net /LED_M4: track 0.00 -> 42.4 mm, vias 0 -> 1
- net /DATA: track 0.00 -> 41.8 mm
- net /LED_ANS_TRUE: track 23.6 -> 65.0 mm
- net /LED_ANS_A: track 44.9 -> 83.7 mm
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- added copper zone on B.Cu, net (none)
- added copper zone on F.Cu, net (none)
Other:
- board outline added: 108.7 x 94 mm
