File: stm32f401nucl/piko_stm32f4nucl/piko_stm32f4nucl.kicad_pcb (KiCad board)
At the start: 2 copper layers, 108.7 x 94 mm, 35 parts, among them J1 Micro_SD_Card_Det, U1 NUCLEO-64

Commit message: mmc not reply
Connections:
- net Net-(J1-Pad1) renamed /DAT2
- net Net-(J1-Pad8) renamed /DAT1
