File: circuit/test_2/end_stm32f401re.kicad_pcb (KiCad board)
At the start: 2 copper layers, 37 parts, among them J1 Micro_SD_Card_Det, J2 USB_B_Micro, U1 MAX98357_DAC, U2 STM32F401RETx, U3 AMS1117-3.3

Commit message: test 2 ok
Parts:
- moved C-XTAL1 128.7 mm to (74.6, 66.2), turned to 270 degrees
- moved Y-XTAL1 126.5 mm to (72.5, 70.8), turned to 90 degrees
- moved C-XTAL2 124.7 mm to (74.6, 70.3), turned to 90 degrees
- moved D-ANS1 112.3 mm to (88.7, 74.3), turned to 0 degrees
- moved R-RST1 103.6 mm to (74.4, 57.8)
- moved SW-RST1 103.6 mm to (71.2, 55.1)
- moved SW-ANS1 103.4 mm to (85.9, 83.3), turned to 0 degrees
- moved SW-ANS2 100.6 mm to (100.2, 83.1), turned to 0 degrees
- moved J-SWD1 98.6 mm to (92.8, 37.7), turned to 90 degrees
- moved D-BTN1 98.1 mm to (88.7, 77.9)
- moved D-BTN2 97.8 mm to (103.9, 77.6)
- moved RL-BTN1 97.5 mm to (96.5, 78.8), turned to 180 degrees
- moved C-ANS1 97.1 mm to (89.1, 87.8), turned to 180 degrees
- moved RL-ANS1 97.1 mm to (96.6, 73.7), turned to 0 degrees
- moved R-ANS1 96.8 mm to (89.1, 84.4), turned to 180 degrees
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Connections:
- J-VREG1 pad 1: VDD -> VCC
- J-VREG1 pad 2: VCC -> VDD
- J2 pad 1: VCC -> Net-(J2-Pad1)
- U2 pad 46: Net-(U2-Pad46) -> /SW_DIO
- U2 pad 49: Net-(U2-Pad49) -> /SW_CLK
- U2 pad 60: Net-(U2-Pad60) -> GND
Routing:
- net GND: track 32.4 -> 413.4 mm, vias 0 -> 4
- net VDD: track 0.00 -> 296.0 mm, vias 0 -> 12
- net /DAC_DIN: track 0.00 -> 72.9 mm, vias 0 -> 1
- net /BTN_B: track 13.3 -> 78.7 mm, vias 0 -> 1
- net /NRST: track 8.26 -> 69.3 mm, vias 0 -> 1
- net /DAC_BCLK: track 0.00 -> 55.3 mm, vias 0 -> 1
- net /DAC_LRC: track 0.00 -> 46.9 mm, vias 0 -> 1
- net /MMC_MISO: track 0.00 -> 43.3 mm, vias 0 -> 1
- net /BTN_A: track 12.9 -> 55.4 mm, vias 0 -> 1
- net /SW_DIO: track 0.00 -> 31.9 mm, vias 0 -> 1
- net /MMC_NSS: track 0.00 -> 29.3 mm
- net Net-(C-XTAL2-Pad1): track 2.48 -> 31.5 mm, vias 0 -> 1
- net /MMC_MOSI: track 0.00 -> 27.7 mm, vias 0 -> 2
- net /MMC_SCK: track 0.00 -> 26.5 mm
- net Net-(C-XTAL1-Pad1): track 2.49 -> 27.8 mm, vias 0 -> 1
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- added copper zone on B.Cu, net (none)
- added copper zone on F.Cu, net (none)
Other:
- board outline added: 70 x 55.8 mm
- net class Default: via_dia 2 -> 1.6

Commit message: test 2 progress
Changed lines of the file:
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@@
     (thickness 1.6)
     (drawings 5)
-    (tracks 634)
+    (tracks 632)
     (zones 0)
     (modules 37)
@@
   (segment (start 128.644999 80.455001) (end 128.7 80.4) (width 0.6) (layer F.Cu) (net 16))
   (segment (start 123.395001 80.455001) (end 128.644999 80.455001) (width 0.6) (layer F.Cu) (net 16))
-  (segment (start 120.742111 36.261391) (end 121.103502 35.9) (width 0.4) (layer B.Cu) (net 16))
-  (segment (start 120.742111 37.511391) (end 120.742111 36.261391) (width 0.4) (layer B.Cu) (net 16))
-  (segment (start 121.103502 35.9) (end 125.4 35.9) (width 0.4) (layer B.Cu) (net 16))
-  (segment (start 125.4 35.9) (end 125.8 36.3) (width 0.4) (layer B.Cu) (net 16))
-  (segment (start 125.822111 36.30931) (end 125.822111 37.511391) (width 0.4) (layer B.Cu) (net 16))
-  (segment (start 125.812801 36.3) (end 125.822111 36.30931) (width 0.4) (layer B.Cu) (net 16))
-  (segment (start 125.8 36.3) (end 125.812801 36.3) (width 0.4) (layer B.Cu) (net 16))
   (via (at 114.4 82.6) (size 1.6) (drill 0.8) (layers F.Cu B.Cu) (net 16))
   (segment (start 113.1 81.3) (end 114.4 82.6) (width 0.6) (layer B.Cu) (net 16))
@@
   (segment (start 103.1 44.9) (end 107.4 44.9) (width 0.4) (layer F.Cu) (net 16))
   (segment (start 102.2 44) (end 103.1 44.9) (width 0.4) (layer F.Cu) (net 16))
+  (segment (start 120.742111 36.261391) (end 121.103502 35.9) (width 0.4) (layer B.Cu) (net 16))
+  (segment (start 120.742111 37.511391) (end 120.742111 36.261391) (width 0.4) (layer B.Cu) (net 16))
+  (segment (start 121.103502 35.9) (end 125.5 35.9) (width 0.4) (layer B.Cu) (net 16))
+  (segment (start 125.822111 36.222111) (end 125.822111 37.511391) (width 0.4) (layer B.Cu) (net 16))
+  (segment (start 125.5 35.9) (end 125.822111 36.222111) (width 0.4) (layer B.Cu) (net 16))
   (segment (start 105.03 56.005) (end 105.03 51.23) (width 0.3) (layer F.Cu) (net 17))
   (segment (start 105.03 51.23) (end 99.7 45.9) (width 0.3) (layer F.Cu) (net 17))
