File: circuit/test_2/end_stm32f401re.sch (KiCad schematic (older format))
At the start: 37 parts, among them J1 Micro_SD_Card_Det, J2 USB_B_Micro, U1 MAX98357_DAC, U2 STM32F401RETx, U3 AMS1117-3.3

Commit message: test 2 ok
Connections:
- net GND: now also U2.60 (BOOT0)
- net SW_CLK: now also U2.49 (PA14)
- net SW_DIO: now also U2.46 (PA13)
- net VCC: now also J-VREG1.1 (Pin_1); no longer J-VREG1.2 (Pin_2), J2.1 (VBUS)
- net VDD: now also J-VREG1.2 (Pin_2); no longer J-VREG1.1 (Pin_1)
Changed lines of the file:
@@
 $EndComp
-$Comp
-L power:VCC #PWR0110
-U 1 1 5E1B86C3
-P 3750 3450
-F 0 "#PWR0110" H 3750 3300 50  0001 C CNN
-F 1 "VCC" H 3767 3623 50  0000 C CNN
-F 2 "" H 3750 3450 50  0001 C CNN
-F 3 "" H 3750 3450 50  0001 C CNN
-	1    3750 3450
-	1    0    0    -1
-$EndComp
-Wire Wire Line
-	3850 3450 3750 3450
 $Comp
 L power:GND #PWR0111
@@
 L power:VDD #PWR0112
 U 1 1 5E1EE69F
-P 5600 3650
-F 0 "#PWR0112" H 5600 3500 50  0001 C CNN
-F 1 "VDD" H 5617 3823 50  0000 C CNN
-F 2 "" H 5600 3650 50  0001 C CNN
-F 3 "" H 5600 3650 50  0001 C CNN
-	1    5600 3650
+P 5700 3650
+F 0 "#PWR0112" H 5700 3500 50  0001 C CNN
+F 1 "VDD" H 5717 3823 50  0000 C CNN
+F 2 "" H 5700 3650 50  0001 C CNN
+F 3 "" H 5700 3650 50  0001 C CNN
+	1    5700 3650
 	1    0    0    -1
 $EndComp
@@
 L power:VCC #PWR0113
 U 1 1 5E1EF094
-P 5700 3650
-F 0 "#PWR0113" H 5700 3500 50  0001 C CNN
-F 1 "VCC" H 5717 3823 50  0000 C CNN
-F 2 "" H 5700 3650 50  0001 C CNN
-F 3 "" H 5700 3650 50  0001 C CNN
-	1    5700 3650
+P 5600 3650
+F 0 "#PWR0113" H 5600 3500 50  0001 C CNN
+F 1 "VCC" H 5617 3823 50  0000 C CNN
+F 2 "" H 5600 3650 50  0001 C CNN
+F 3 "" H 5600 3650 50  0001 C CNN
+	1    5600 3650
 	1    0    0    -1
 $EndComp
@@
 Text Label 6150 3400 0    50   ~ 0
 BTN_B
+Wire Wire Line
+	7750 3000 8050 3000
+Wire Wire Line
+	7750 3100 8050 3100
+Text Label 8050 3000 0    50   ~ 0
+SW_DIO
+Text Label 8050 3100 0    50   ~ 0
+SW_CLK
+$Comp
+L power:GND #PWR?
+U 1 1 5E190E0F
+P 6300 1900
+F 0 "#PWR?" H 6300 1650 50  0001 C CNN
+F 1 "GND" H 6305 1727 50  0000 C CNN
+F 2 "" H 6300 1900 50  0001 C CNN
+F 3 "" H 6300 1900 50  0001 C CNN
+	1    6300 1900
+	1    0    0    -1
+$EndComp
+Wire Wire Line
+	6450 1900 6300 1900
 $EndSCHEMATC

Commit message: test 2 progress
Changed lines of the file:
@@
 L power:VDD #PWR015
 U 1 1 5DFA14F3
-P 3450 4450
-F 0 "#PWR015" H 3450 4300 50  0001 C CNN
-F 1 "VDD" H 3467 4623 50  0000 C CNN
-F 2 "" H 3450 4450 50  0001 C CNN
-F 3 "" H 3450 4450 50  0001 C CNN
-	1    3450 4450
-	1    0    0    -1
-$EndComp
-Wire Wire Line
-	3750 4450 3450 4450
-Wire Wire Line
-	3200 4450 3450 4450
-Wire Wire Line
-	3200 4450 3200 4650
-Connection ~ 3450 4450
+P 3750 4350
+F 0 "#PWR015" H 3750 4200 50  0001 C CNN
+F 1 "VDD" H 3767 4523 50  0000 C CNN
+F 2 "" H 3750 4350 50  0001 C CNN
+F 3 "" H 3750 4350 50  0001 C CNN
+	1    3750 4350
+	1    0    0    -1
+$EndComp
 Wire Wire Line
 	3200 4800 3000 4800
@@
 SW_CLK
 $Comp
-L power:GND #PWR?
+L power:GND #PWR0110
 U 1 1 5E190E0F
 P 6300 1900
-F 0 "#PWR?" H 6300 1650 50  0001 C CNN
+F 0 "#PWR0110" H 6300 1650 50  0001 C CNN
 F 1 "GND" H 6305 1727 50  0000 C CNN
 F 2 "" H 6300 1900 50  0001 C CNN
@@
 Wire Wire Line
 	6450 1900 6300 1900
+Wire Wire Line
+	3750 4350 3750 4450
+$Comp
+L power:VDD #PWR?
+U 1 1 5E150C29
+P 3000 4650
+F 0 "#PWR?" H 3000 4500 50  0001 C CNN
+F 1 "VDD" H 3017 4823 50  0000 C CNN
+F 2 "" H 3000 4650 50  0001 C CNN
+F 3 "" H 3000 4650 50  0001 C CNN
+	1    3000 4650
+	1    0    0    -1
+$EndComp
+Wire Wire Line
+	3200 4650 3000 4650
 $EndSCHEMATC

Commit message: add diode on power reg
Parts:
- added D-VREG1: D, Diode_SMD:D_SMA_Handsoldering, symbol Device:D
Connections:
- wire segments 140 -> 142
Other:
- moved on the sheet: C-VREG2
Changed lines of the file:
@@
 L power:VDD #PWR0108
 U 1 1 5E1AC6BA
-P 6050 5650
-F 0 "#PWR0108" H 6050 5500 50  0001 C CNN
-F 1 "VDD" H 6067 5823 50  0000 C CNN
-F 2 "" H 6050 5650 50  0001 C CNN
-F 3 "" H 6050 5650 50  0001 C CNN
-	1    6050 5650
+P 6350 5600
+F 0 "#PWR0108" H 6350 5450 50  0001 C CNN
+F 1 "VDD" H 6367 5773 50  0000 C CNN
+F 2 "" H 6350 5600 50  0001 C CNN
+F 3 "" H 6350 5600 50  0001 C CNN
+	1    6350 5600
 	1    0    0    -1
 $EndComp
@@
 L Device:C C-VREG2
 U 1 1 5E1BF4DE
-P 6050 5850
-F 0 "C-VREG2" H 6165 5896 50  0000 L CNN
-F 1 "C" H 6165 5805 50  0000 L CNN
-F 2 "Capacitor_SMD:C_0805_2012Metric_Pad1.15x1.40mm_HandSolder" H 6088 5700 50  0001 C CNN
-F 3 "~" H 6050 5850 50  0001 C CNN
-	1    6050 5850
+P 6350 5850
+F 0 "C-VREG2" H 6465 5896 50  0000 L CNN
+F 1 "C" H 6465 5805 50  0000 L CNN
+F 2 "Capacitor_SMD:C_0805_2012Metric_Pad1.15x1.40mm_HandSolder" H 6388 5700 50  0001 C CNN
+F 3 "~" H 6350 5850 50  0001 C CNN
+	1    6350 5850
 	1    0    0    -1
 $EndComp
@@
 Connection ~ 5650 6000
 Wire Wire Line
-	5650 6000 6050 6000
-Wire Wire Line
 	5650 6050 5650 6000
 Wire Wire Line
@@
 	5250 5700 5250 5650
 Connection ~ 5250 5650
-Wire Wire Line
-	5950 5650 6050 5650
-Wire Wire Line
-	6050 5700 6050 5650
-Connection ~ 6050 5650
 $Comp
 L Connector:Conn_01x03_Male J-VREG1
@@
 	3750 4350 3750 4450
 $Comp
-L power:VDD #PWR?
+L power:VDD #PWR0115
 U 1 1 5E150C29
 P 3000 4650
-F 0 "#PWR?" H 3000 4500 50  0001 C CNN
+F 0 "#PWR0115" H 3000 4500 50  0001 C CNN
 F 1 "VDD" H 3017 4823 50  0000 C CNN
 F 2 "" H 3000 4650 50  0001 C CNN
@@
 Wire Wire Line
 	3200 4650 3000 4650
+$Comp
+L Device:D D-VREG1
+U 1 1 5E160CA1
+P 6150 5650
+F 0 "D-VREG1" H 6150 5434 50  0000 C CNN
+F 1 "D" H 6150 5525 50  0000 C CNN
+F 2 "Diode_SMD:D_SMA_Handsoldering" H 6150 5650 50  0001 C CNN
+F 3 "~" H 6150 5650 50  0001 C CNN
+	1    6150 5650
+	-1   0    0    1
+$EndComp
+Wire Wire Line
+	6350 6000 5650 6000
+Wire Wire Line
+	5950 5650 6000 5650
+Wire Wire Line
+	6350 5600 6350 5650
+Wire Wire Line
+	6300 5650 6350 5650
+Connection ~ 6350 5650
+Wire Wire Line
+	6350 5650 6350 5700
 $EndSCHEMATC

Commit message: RESET to START
Parts:
- removed SW-RST1: SW_Push, Button_Switch_THT:SW_PUSH_6mm, symbol Switch:SW_Push
- added C-START1: C, Capacitor_SMD:C_0805_2012Metric_Pad1.15x1.40mm_HandSolder, symbol Device:C
- added R-START1: 10K, Resistor_SMD:R_0805_2012Metric_Pad1.15x1.40mm_HandSolder, symbol Device:R
- added SW-START1: SW_Push, Button_Switch_THT:SW_PUSH_6mm, symbol Switch:SW_Push
Connections:
- net labels added: BTN_START
- wire segments 142 -> 150
Changed lines of the file:
@@
 $EndComp
-Wire Wire Line
-	6450 1600 6450 1700
-$Comp
-L Switch:SW_Push SW-RST1
-U 1 1 5DFDB8B6
-P 6200 1700
-F 0 "SW-RST1" H 6200 1985 50  0000 C CNN
-F 1 "SW_Push" H 6200 1894 50  0000 C CNN
-F 2 "Button_Switch_THT:SW_PUSH_6mm" H 6200 1900 50  0001 C CNN
-F 3 "" H 6200 1900 50  0001 C CNN
-	1    6200 1700
-	1    0    0    -1
-$EndComp
-Wire Wire Line
-	6400 1700 6450 1700
-Connection ~ 6450 1700
-$Comp
-L power:GND #PWR0104
-U 1 1 5DFDDEEE
-P 5900 1700
-F 0 "#PWR0104" H 5900 1450 50  0001 C CNN
-F 1 "GND" H 5905 1527 50  0000 C CNN
-F 2 "" H 5900 1700 50  0001 C CNN
-F 3 "" H 5900 1700 50  0001 C CNN
-	1    5900 1700
-	1    0    0    -1
-$EndComp
-Wire Wire Line
-	6000 1700 5900 1700
 Wire Wire Line
 	6150 4300 6450 4300
@@
 Text Label 5250 2150 0    50   ~ 0
 SW_DIO
-Wire Wire Line
-	6450 1700 6450 1750
-Text Label 6450 1750 0    50   ~ 0
-NRST
 Text Label 5250 2250 0    50   ~ 0
 NRST
@@
 Wire Wire Line
 	6350 5650 6350 5700
+Wire Wire Line
+	6450 4600 6150 4600
+Text Label 6150 4600 0    50   ~ 0
+BTN_START
+Wire Wire Line
+	6450 1600 6450 1700
+$Comp
+L Switch:SW_Push SW-START1
+U 1 1 5E250FBA
+P 2100 5950
+F 0 "SW-START1" H 2100 6235 50  0000 C CNN
+F 1 "SW_Push" H 2100 6144 50  0000 C CNN
+F 2 "Button_Switch_THT:SW_PUSH_6mm" H 2100 6150 50  0001 C CNN
+F 3 "" H 2100 6150 50  0001 C CNN
+	1    2100 5950
+	1    0    0    -1
+$EndComp
+$Comp
+L Device:R R-START1
+U 1 1 5E250FC0
+P 1850 5750
+F 0 "R-START1" H 1920 5796 50  0000 L CNN
+F 1 "10K" H 1920 5705 50  0000 L CNN
+F 2 "Resistor_SMD:R_0805_2012Metric_Pad1.15x1.40mm_HandSolder" V 1780 5750 50  0001 C CNN
+F 3 "~" H 1850 5750 50  0001 C CNN
+	1    1850 5750
+	1    0    0    -1
+$EndComp
+Wire Wire Line
+	1900 5950 1850 5950
+Wire Wire Line
+	1850 5950 1850 5900
+Wire Wire Line
+	1850 5950 1750 5950
+Connection ~ 1850 5950
+$Comp
+L Device:C C-START1
+U 1 1 5E250FCA
+P 2100 6100
+F 0 "C-START1" V 1848 6100 50  0000 C CNN
+F 1 "C" V 1939 6100 50  0000 C CNN
+F 2 "Capacitor_SMD:C_0805_2012Metric_Pad1.15x1.40mm_HandSolder" H 2138 5950 50  0001 C CNN
+F 3 "~" H 2100 6100 50  0001 C CNN
+	1    2100 6100
+	0    1    1    0
+$EndComp
+$Comp
+L power:GND #PWR0104
+U 1 1 5E250FD0
+P 2350 6100
+F 0 "#PWR0104" H 2350 5850 50  0001 C CNN
+F 1 "GND" H 2355 5927 50  0000 C CNN
+F 2 "" H 2350 6100 50  0001 C CNN
+F 3 "" H 2350 6100 50  0001 C CNN
+	1    2350 6100
+	1    0    0    -1
+$EndComp
+$Comp
+L power:VDD #PWR0116
+U 1 1 5E250FD6
+P 1850 5550
+F 0 "#PWR0116" H 1850 5400 50  0001 C CNN
+F 1 "VDD" H 1867 5723 50  0000 C CNN
+F 2 "" H 1850 5550 50  0001 C CNN
+F 3 "" H 1850 5550 50  0001 C CNN
+	1    1850 5550
+	1    0    0    -1
+$EndComp
+Wire Wire Line
+	2300 5950 2350 5950
+Wire Wire Line
+	2350 5950 2350 6100
+Wire Wire Line
+	2250 6100 2350 6100
+Connection ~ 2350 6100
+Wire Wire Line
+	1950 6100 1850 6100
+Wire Wire Line
+	1850 6100 1850 5950
+Wire Wire Line
+	1850 5550 1850 5600
+Text Label 1750 5950 0    50   ~ 0
+BTN_START
+Wire Wire Line
+	6450 1700 6300 1700
+Connection ~ 6450 1700
+Text Label 6300 1700 0    50   ~ 0
+NRST
 $EndSCHEMATC
